Commit message: 1.15

File: install/rm_gimbal_description/share/rm_gimbal_description/urdf/rm_gimbal.urdf.xacro (robot description, xacro)
@@ -1,25 +1 @@
-<?xml version="1.0" encoding="utf-8"?>
-<robot name="rm_gimbal"
-  xmlns:xacro="http://ros.org/wiki/xacro">
-  <xacro:arg name="xyz" default="0.00 0 0.042" />
-  <xacro:arg name="rpy" default="0 0 0" />
-  <link name="odom" />
-  <link name="gimbal_link" />
-  <joint name="gimbal_joint" type="floating">
-    <parent link="odom" />
-    <child link="gimbal_link" />
-  </joint>
-  <link name="camera_link" />
-  <joint name="camera_joint" type="fixed">
-    <origin xyz="$(arg xyz)" rpy="$(arg rpy)" />
-    <parent link="gimbal_link" />
-    <child link="camera_link" />
-    <axis xyz="0 0 0" />
-  </joint>
-  <link name="camera_optical_frame" />
-  <joint name="camera_optical_joint" type="fixed">
-    <origin xyz="0 0 0" rpy="${-pi/2} 0 ${-pi/2}" />
-    <parent link="camera_link" />
-    <child link="camera_optical_frame" />
-  </joint>
-</robot>
+/home/mechax/zyb/mechax_cv_trajectory/src/rm_gimbal_description/urdf/rm_gimbal.urdf.xacro

File: src/rm_gimbal_description/urdf/rm_gimbal.urdf.xacro (robot description, xacro)
@@ -2,6 +2,6 @@
 <robot name="rm_gimbal"
   xmlns:xacro="http://ros.org/wiki/xacro">
-  <xacro:arg name="xyz" default="0.00 0 0.042" />
-  <xacro:arg name="rpy" default="0 0 0" />
+  <xacro:arg name="xyz" default="0.00 0.060 0.042" />
+  <xacro:arg name="rpy" default="0 ${pi/2} 0" />
   <link name="odom" />
   <link name="gimbal_link" />

Commit message: 2024.2.27

File: install/rm_gimbal_description/share/rm_gimbal_description/urdf/rm_gimbal.urdf.xacro (robot description, xacro)
@@ -2,6 +2,4 @@
 <robot name="rm_gimbal"
   xmlns:xacro="http://ros.org/wiki/xacro">
-  <xacro:arg name="xyz" default="0.080 0.000 0.030" />
-  <xacro:arg name="rpy" default="0 0 0" />
   <link name="odom" />
   <link name="gimbal_link" />
@@ -12,5 +10,5 @@
   <link name="camera_link" />
   <joint name="camera_joint" type="fixed">
-    <origin xyz="$(arg xyz)" rpy="$(arg rpy)" />
+    <origin xyz="0.080 0.000 0.04" rpy="0 0.0 ${pi/32}" />
     <parent link="gimbal_link" />
     <child link="camera_link" />
@@ -23,3 +21,8 @@
     <child link="camera_optical_frame" />
   </joint>
+  <link name="horizom_gimbal_link" />
+  <joint name="horizom_gimbal_joint" type="floating">
+    <parent link = "gimbal_link" />
+    <child link = "horizom_gimbal_link" />
+  </joint>
 </robot>

Commit message: 2024.3.8

File: install/rm_gimbal_description/share/rm_gimbal_description/urdf/rm_gimbal.urdf.xacro (robot description, xacro)
@@ -26,3 +26,21 @@
     <child link = "horizom_gimbal_link" />
   </joint>
+  <link name="prediction_gimbal_link" />
+  <joint name="prediction_gimbal_joint" type= "floating">
+    <parent link = "horizom_gimbal_link" />
+    <child link = "prediction_gimbal_link" />
+  </joint>
+  <link name="prediction_camera_link" />
+  <joint name="prediction_camera_joint" type="fixed">
+    <origin xyz="0.080 0.000 0.04" rpy="0 0.0 ${pi/32}" />
+    <parent link="prediction_gimbal_link" />
+    <child link="prediction_camera_link" />
+    <axis xyz="0 0 0" />
+  </joint>
+  <link name="prediction_camera_optical_frame" />
+  <joint name="prediction_camera_optical_joint" type="fixed">
+    <origin xyz="0 0 0" rpy="${-pi/2} 0 ${-pi/2}" />
+    <parent link="prediction_camera_link" />
+    <child link="prediction_camera_optical_frame" />
+  </joint>
 </robot>
