Commit message: add front and back assist detector

File: src/rm_gimbal_description/urdf/rm_gimbal.urdf.xacro (robot description, xacro)
@@ -2,30 +2,81 @@
 <robot name="rm_gimbal"
   xmlns:xacro="http://ros.org/wiki/xacro">
-  <link name="odom" />
-  <link name="gimbal_link" />
-  <joint name="gimbal_joint" type="fixed">
-    <parent link="odom" />
-    <child link="gimbal_link" />
+  <link name="leftodom" />
+  <link name="left_gimbal_link" />
+  <joint name="left_gimbal_joint" type="fixed">
+    <origin xyz="0.0 0 0" rpy="0 0 0" />
+    <parent link="leftodom" />
+    <child link="left_gimbal_link" />
   </joint>
-  <link name="camera_link" />
-  <joint name="camera_joint" type="fixed">
+  <link name="rightodom" />
+  <link name="right_gimbal_link" />
+  <joint name="right_gimbal_joint" type="fixed">
+    <origin xyz="0.0 0 0" rpy="0 0 0" />
+    <parent link="rightodom" />
+    <child link="right_gimbal_link" />
+  </joint>
+  <link name="bigodom" />
+  <joint name="bigodom_leftodom_joint" type="fixed">
+    <origin xyz="0.10 0 0" rpy="0 0 0" />
+    <parent link="leftodom" />
+    <child link="bigodom" />
+  </joint>
+  <joint name="bigodom_rightodom_link" type="fixed">
+    <origin xyz="0.10 0 0" rpy="0 0 0" />
+    <parent link="bigodom" />
+    <child link="rightodom" />
+  </joint>
+  <link name="big_gimbal_link" />
+  <joint name="big_gimbal_joint" type="fixed">
+    <origin xyz="0.0 0 0" rpy="0 0 0" />
+    <parent link="bigodom" />
+    <child link="big_gimbal_link" />
+  </joint>
+  <link name="front_camera_link"/>
+  <joint name="front_camera_joint" type="fixed">
+    <origin xyz="0 0 0" rpy="0 0 0" />
+    <parent link="big_gimbal_link" />
+    <child link="front_camera_link" />
+  </joint>
+  <link name="front_camera_optical_frame" />
+  <joint name="front_camera_optical_joint" type="fixed">
+    <origin xyz="0 0 0" rpy="${-pi/2} 0 ${-pi/2}" />
+    <parent link="front_camera_link" />
+    <child link="front_camera_optical_frame" />
+  </joint>
+  <link name="back_camera_link" />
+  <joint name="back_camera_joint" type="fixed">
+    <origin xyz="0 0 0" rpy="0 0 0" />
+    <parent link="big_gimbal_link" />
+    <child link="back_camera_link" />
+  </joint>
+  <link name="back_camera_optical_frame" />
+  <joint name="back_camera_optical_joint" type="fixed">
+    <origin xyz="0 0 0" rpy="${-pi/2} 0 ${-pi/2}" />
+    <parent link="back_camera_link" />
+    <child link="back_camera_optical_frame" />
+  </joint>
+  <link name="left_camera_link" />
+  <joint name="left_camera_joint" type="fixed">
     <origin xyz="0.050 0.000 0.040" rpy="0 ${pi/140} -${pi/160}" />
-    <parent link="gimbal_link" />
-    <child link="camera_link" />
+    <parent link="left_gimbal_link" />
+    <child link="left_camera_link" />
     <axis xyz="0 0 0" />
   </joint>
-  <link name="camera_optical_frame" />
-  <joint name="camera_optical_joint" type="fixed">
+  <link name="left_camera_optical_frame" />
+  <joint name="left_camera_optical_joint" type="fixed">
     <origin xyz="0 0 0" rpy="${-pi/2} 0 ${-pi/2}" />
-    <parent link="camera_link" />
-    <child link="camera_optical_frame" />
+    <parent link="left_camera_link" />
+    <child link="left_camera_optical_frame" />
   </joint>
   <link name="horizom_gimbal_link" />
-  <joint name="horizom_gimbal_joint" type="floating">
-    <parent link = "gimbal_link" />
+  <joint name="horizom_gimbal_joint" type="fixed">
+    <origin xyz="0.0 0 0" rpy="0 0 0" />
+    <parent link = "left_gimbal_link" />
     <child link = "horizom_gimbal_link" />
   </joint>
   <link name="prediction_gimbal_link" />
-  <joint name="prediction_gimbal_joint" type="floating">
+  <joint name="prediction_gimbal_joint" type="fixed">
+    <origin xyz="0.0 0 0" rpy="0 0 0" />
     <parent link = "horizom_gimbal_link" />
     <child link = "prediction_gimbal_link" />
@@ -44,9 +95,3 @@
     <child link="prediction_camera_optical_frame" />
   </joint>
-  <link name="bigodom" />
-  <joint name="bigodom_joint" type="fixed">
-    <origin xyz="-0.10 0 0" rpy="0 0 0" />
-    <parent link="odom" />
-    <child link="bigodom" />
-  </joint>
 </robot>

Commit message: change to rm_left_auto_aim

File: src/rm_gimbal_description/urdf/rm_gimbal.urdf.xacro (robot description, xacro)
@@ -70,4 +70,17 @@
     <child link="left_camera_optical_frame" />
   </joint>
+  <link name="right_camera_link" />
+  <joint name="right_camera_joint" type="fixed">
+    <origin xyz="0.050 0.000 0.040" rpy="0 ${pi/140} -${pi/180}" />
+    <parent link="right_gimbal_link" />
+    <child link="right_camera_link" />
+    <axis xyz="0 0 0" />
+  </joint>
+  <link name="right_camera_optical_frame" />
+  <joint name="right_camera_optical_joint" type="fixed">
+    <origin xyz="0 0 0" rpy="${-pi/2} 0 ${-pi/2}" />
+    <parent link="right_camera_link" />
+    <child link="right_camera_optical_frame" />
+  </joint>
   <link name="horizom_gimbal_link" />
   <joint name="horizom_gimbal_joint" type="fixed">

Commit message: 2024.5.7

File: src/rm_gimbal_description/urdf/rm_gimbal.urdf.xacro (robot description, xacro)
@@ -11,6 +11,5 @@
   <link name="rightodom" />
   <link name="right_gimbal_link" />
-  <joint name="right_gimbal_joint" type="fixed">
-    <origin xyz="0.0 0 0" rpy="0 0 0" />
+  <joint name="right_gimbal_joint" type="floating">
     <parent link="rightodom" />
     <child link="right_gimbal_link" />
@@ -18,16 +17,15 @@
   <link name="bigodom" />
   <joint name="bigodom_leftodom_joint" type="fixed">
-    <origin xyz="0.10 0 0" rpy="0 0 0" />
+    <origin xyz="0.00 -0.10 0" rpy="0 0 0" />
     <parent link="leftodom" />
     <child link="bigodom" />
   </joint>
   <joint name="bigodom_rightodom_link" type="fixed">
-    <origin xyz="0.10 0 0" rpy="0 0 0" />
+    <origin xyz="0.0 -0.10 0" rpy="0 0 0" />
     <parent link="bigodom" />
     <child link="rightodom" />
   </joint>
   <link name="big_gimbal_link" />
-  <joint name="big_gimbal_joint" type="fixed">
-    <origin xyz="0.0 0 0" rpy="0 0 0" />
+  <joint name="big_gimbal_joint" type="floating">
     <parent link="bigodom" />
     <child link="big_gimbal_link" />
@@ -47,5 +45,5 @@
   <link name="back_camera_link" />
   <joint name="back_camera_joint" type="fixed">
-    <origin xyz="0 0 0" rpy="0 0 0" />
+    <origin xyz="0 0 0" rpy="0 0 ${pi/2}" />
     <parent link="big_gimbal_link" />
     <child link="back_camera_link" />
@@ -90,6 +88,5 @@
   </joint>
   <link name="prediction_gimbal_link" />
-  <joint name="prediction_gimbal_joint" type="fixed">
-    <origin xyz="0.0 0 0" rpy="0 0 0" />
+  <joint name="prediction_gimbal_joint" type="floating">
     <parent link = "horizom_gimbal_link" />
     <child link = "prediction_gimbal_link" />

Commit message: add outpost

File: src/rm_gimbal_description/urdf/rm_gimbal.urdf.xacro (robot description, xacro)
@@ -4,6 +4,5 @@
   <link name="leftodom" />
   <link name="left_gimbal_link" />
-  <joint name="left_gimbal_joint" type="fixed">
-    <origin xyz="0.0 0 0" rpy="0 0 0" />
+  <joint name="left_gimbal_joint" type="floating">
     <parent link="leftodom" />
     <child link="left_gimbal_link" />
@@ -57,8 +56,7 @@
   <link name="left_camera_link" />
   <joint name="left_camera_joint" type="fixed">
-    <origin xyz="0.050 0.000 0.040" rpy="0 ${pi/140} -${pi/160}" />
+    <origin xyz="0.110 0.045 0.030" rpy="0 0.0 0" />
     <parent link="left_gimbal_link" />
     <child link="left_camera_link" />
-    <axis xyz="0 0 0" />
   </joint>
   <link name="left_camera_optical_frame" />
@@ -73,5 +71,4 @@
     <parent link="right_gimbal_link" />
     <child link="right_camera_link" />
-    <axis xyz="0 0 0" />
   </joint>
   <link name="right_camera_optical_frame" />

Commit message: higher fps

File: src/rm_gimbal_description/urdf/rm_gimbal.urdf.xacro (robot description, xacro)
@@ -1,5 +1,4 @@
 <?xml version="1.0" encoding="utf-8"?>
-<robot name="rm_gimbal"
-  xmlns:xacro="http://ros.org/wiki/xacro">
+<robot name="rm_gimbal" xmlns:xacro="http://ros.org/wiki/xacro">
   <link name="leftodom" />
   <link name="left_gimbal_link" />
@@ -56,5 +55,5 @@
   <link name="left_camera_link" />
   <joint name="left_camera_joint" type="fixed">
-    <origin xyz="0.110 0.045 0.030" rpy="0 0.0 0" />
+    <origin xyz="0.0481 0.00 0.047" rpy="0 ${pi/360} ${pi/360}" />
     <parent link="left_gimbal_link" />
     <child link="left_camera_link" />
@@ -68,5 +67,5 @@
   <link name="right_camera_link" />
   <joint name="right_camera_joint" type="fixed">
-    <origin xyz="0.050 0.000 0.040" rpy="0 ${pi/140} -${pi/180}" />
+    <origin xyz="0.050 0.000 0.040" rpy="0 0 -${pi/180}" />
     <parent link="right_gimbal_link" />
     <child link="right_camera_link" />
@@ -78,27 +77,3 @@
     <child link="right_camera_optical_frame" />
   </joint>
-  <link name="horizom_gimbal_link" />
-  <joint name="horizom_gimbal_joint" type="fixed">
-    <origin xyz="0.0 0 0" rpy="0 0 0" />
-    <parent link = "left_gimbal_link" />
-    <child link = "horizom_gimbal_link" />
-  </joint>
-  <link name="prediction_gimbal_link" />
-  <joint name="prediction_gimbal_joint" type="floating">
-    <parent link = "horizom_gimbal_link" />
-    <child link = "prediction_gimbal_link" />
-  </joint>
-  <link name="prediction_camera_link" />
-  <joint name="prediction_camera_joint" type="fixed">
-    <origin xyz="0.050 0.000 0.040" rpy="0 ${pi/140} -${pi/180}" />
-    <parent link="prediction_gimbal_link" />
-    <child link="prediction_camera_link" />
-    <axis xyz="0 0 0" />
-  </joint>
-  <link name="prediction_camera_optical_frame" />
-  <joint name="prediction_camera_optical_joint" type="fixed">
-    <origin xyz="0 0 0" rpy="${-pi/2} 0 ${-pi/2}" />
-    <parent link="prediction_camera_link" />
-    <child link="prediction_camera_optical_frame" />
-  </joint>
 </robot>

Commit message: optimization

File: src/rm_gimbal_description/urdf/rm_gimbal.urdf.xacro (robot description, xacro)
@@ -4,5 +4,5 @@
   <link name="odom" />
   <link name="gimbal_link" />
-  <joint name="gimbal_joint" type="fixed">
+  <joint name="gimbal_joint" type="floating">
     <parent link="odom" />
     <child link="gimbal_link" />

Commit message: optimization

File: src/rm_gimbal_description/urdf/rm_gimbal.urdf.xacro (robot description, xacro)
@@ -4,5 +4,5 @@
   <link name="odom" />
   <link name="gimbal_link" />
-  <joint name="gimbal_joint" type="fixed">
+  <joint name="gimbal_joint" type="floating">
     <parent link="odom" />
     <child link="gimbal_link" />
@@ -10,8 +10,7 @@
   <link name="camera_link" />
   <joint name="camera_joint" type="fixed">
-    <origin xyz="0.080 0.000 0.04" rpy="0 0.0 ${pi/32}" />
+    <origin xyz="0.070 0.000 0.04" rpy="0 -${pi/180} -${pi/180}" />
     <parent link="gimbal_link" />
     <child link="camera_link" />
-    <axis xyz="0 0 0" />
   </joint>
   <link name="camera_optical_frame" />

Commit message: optimiation

File: src/rm_gimbal_description/urdf/rm_gimbal.urdf.xacro (robot description, xacro)
@@ -55,5 +55,5 @@
   <link name="left_camera_link" />
   <joint name="left_camera_joint" type="fixed">
-    <origin xyz="0.0481 0.00 0.047" rpy="0 ${pi/360} ${pi/360}" />
+    <origin xyz="0.0481 0.00 0.047" rpy="0 ${pi/360} ${pi/180}" />
     <parent link="left_gimbal_link" />
     <child link="left_camera_link" />

Commit message: optimization

File: src/rm_gimbal_description/urdf/rm_gimbal.urdf.xacro (robot description, xacro)
@@ -10,5 +10,5 @@
   <link name="camera_link" />
   <joint name="camera_joint" type="fixed">
-    <origin xyz="0.070 0.000 0.04" rpy="0 -${pi/180} -${pi/180}" />
+    <origin xyz="0.085 0.000  0.035" rpy="0.0  0.0  ${pi / 360}" />
     <parent link="gimbal_link" />
     <child link="camera_link" />

Commit message: optimization

File: src/rm_gimbal_description/urdf/rm_gimbal.urdf.xacro (robot description, xacro)
@@ -10,5 +10,5 @@
   <link name="camera_link" />
   <joint name="camera_joint" type="fixed">
-    <origin xyz="0.085 0.000  0.035" rpy="0.0  0.0  ${pi / 360}" />
+    <origin xyz="0.085 0.000  0.035" rpy="0.0  ${pi / 360}  ${pi / 120}" />
     <parent link="gimbal_link" />
     <child link="camera_link" />

Commit message: init

File: src/rm_gimbal_description/urdf/rm_gimbal.urdf.xacro (robot description, xacro)
@@ -31,3 +31,4 @@
     <parent link="camera_assistant_link" />
     <child link="camera_assistant_optical_frame" />
+  </joint>
 </robot>
